File: kicad/bldc_project.kicad_pcb (KiCad board)
At the start: 4 copper layers, 115 x 60 mm, 155 parts, among them J1 Conn_ARM_SWD_TagConnect_TC203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, J2 Screw_Terminal_01x03, J3 Screw_Terminal_01x03, J4 TYPE-C-31-M-12, Q1 IRFZ44N, Q2 IRFZ44N, Q3 IRFZ44N, Q4 IRFZ44N, Q5 IRFZ44N, Q6 IRFZ44N, Q7 BC847BW,115, SW1 SW_Push, U1 ir2104, U10 MC34063AD, U11 MC34063AD, U14 XC6206P332MR-G, U2 ir2104, U3 ir2104, U4 INA180A2, U5 INA180A2, U6 INA180A2, U7 STM32F303CBTx, Y1 8 MHz

Commit message: [kicad] Layout, mostly power traces + HS signal traces
Parts:
- added H5: MountingHole, bldc:MountingHole_1.152mm_jlcpcb, F.Cu at (1.23, 1.23)
- moved U9 5.81 mm to (55.8, 91.9)
Connections:
- net Net-(U10-DC) renamed /POWER/VBUCK5_IN
- net Net-(U11-DC) renamed /POWER/VBUCK10_IN
- net USB_DM renamed USB_DN
Routing:
- net USB_DN: track 0.00 -> 21.8 mm
- net USB_DP: track 0.00 -> 20.3 mm
- net GND: track 7.64 -> 27.6 mm, vias 0 -> 13
- net +3.3V: track 48.0 -> 65.6 mm
- net /CPU/CAN_L: track 0.00 -> 10.0 mm
- net /CPU/CAN_H: track 0.00 -> 9.30 mm
- net /POWER/VBUCK5_IN: track 0.00 -> 8.63 mm
- net +10V: track 10.7 -> 3.17 mm
- net /CPU/CAN_N: track 0.00 -> 6.18 mm, vias 0 -> 3
- net /POWER/VBUCK5_OUT: track 0.00 -> 3.60 mm
- net USB_VBUS: track 0.00 -> 3.35 mm
- net Net-(U13-PR1): track 0.00 -> 3.06 mm
- net PhaseV_SWITCH: track 3.74 -> 6.60 mm, vias 1 -> 2
- net PhaseV_SD: track 0.00 -> 2.49 mm, vias 0 -> 1
- net PhaseU_SWITCH: track 2.77 -> 5.23 mm, vias 1 -> 2
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- added copper zone on F.Cu, net +10V
- added copper zone on F.Cu, net +3.3V
- added copper zone on F.Cu, net +BATT
- added copper zone on F.Cu, net /POWER/VBUCK10_IN
- added copper zone on F.Cu, net /POWER/VBUCK5_IN
