File: kicad/driver.kicad_sch (KiCad schematic)
At the start: 85 parts, among them Q1 IRFZ44NPBF, Q2 IRFZ44NPBF, Q3 IRFZ44NPBF, Q4 IRFZ44NPBF, Q5 IRFZ44NPBF, Q6 IRFZ44NPBF, U1 ir2104, U2 ir2104, U3 ir2104, U4 INA180A2IDBVR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

Commit message: Exchanged button, 0.33 ohm resistor and 3-pin connectors with cheaper variants
Parts:
- C1, C2, C3: MFR.Part CL21A475KAQNNNE -> (none); Manufacturing part number (none) -> CL21A475KAQNNNE; jlcpcb C1779 -> (none); jlcpcb part number (none) -> C1779
- C10, C11, C12, C13, C14, C15, C7, C8, C9: MFR.Part CL05B103KB5NNNC -> (none); Manufacturing part number (none) -> CL05B103KB5NNNC; jlcpcb C15195 -> (none); jlcpcb part number (none) -> C15195
- C16, C17, C18: MFR.Part ERS1HM471G20OT -> (none); Manufacturing part number (none) -> ERS1HM471G20OT; jlcpcb C106666 -> (none); jlcpcb part number (none) -> C106666
- C19, C20, C21: MFR.Part CL05B104KB54PNC -> (none); Manufacturing part number (none) -> CL05B104KB54PNC; jlcpcb C307331 -> (none); jlcpcb part number (none) -> C307331
- C4, C5, C6: MFR.Part CL10A475KO8NNNC -> (none); Manufacturing part number (none) -> CL10A475KO8NNNC; jlcpcb C19666 -> (none); jlcpcb part number (none) -> C19666
- D1, D2, D3: MFR.Part 1N5819WS -> (none); Manufacturing part number (none) -> 1N5819WS; jlcpcb C191023 -> (none); jlcpcb part number (none) -> C191023
- Q1, Q2, Q3, Q4, Q5, Q6: MFR.Part IRFZ44NPBF -> (none); Manufacturing part number (none) -> IRFZ44NPBF; jlcpcb C2586 -> (none); jlcpcb part number (none) -> C2586
- R1, R2, R3: MFR.Part 1206W4F100JT5E -> (none); Manufacturing part number (none) -> 1206W4F100JT5E; jlcpcb C17903 -> (none); jlcpcb part number (none) -> C17903
- R10, R11, R12: MFR.Part LR2512D-2W-3mR-1% -> (none); Manufacturing part number (none) -> LR2512D-2W-3mR-1%; jlcpcb C500615 -> (none); jlcpcb part number (none) -> C500615
- R13, R14, R15, R16, R17, R18, R19, R20, R21: MFR.Part 0603WAF100KT5E -> (none); Manufacturing part number (none) -> 0603WAF100KT5E; jlcpcb C22936 -> (none); jlcpcb part number (none) -> C22936
- R22, R23, R24, R25, R26, R27, R28, R29, R30, R31, R32, R33: MFR.Part 0603WAF3302T5E -> (none); Manufacturing part number (none) -> 0603WAF3302T5E; jlcpcb C4216 -> (none); jlcpcb part number (none) -> C4216
- R4, R5, R6, R7, R8, R9: MFR.Part 1206W4F510JT5E -> (none); Manufacturing part number (none) -> 1206W4F510JT5E; jlcpcb C18019 -> (none); jlcpcb part number (none) -> C18019
- U1, U2, U3: MFR.Part IR2104STRPBF-JSM -> (none); Manufacturing part number (none) -> IR2104STRPBF-JSM; jlcpcb C5804631 -> (none); jlcpcb part number (none) -> C5804631
- U4, U5, U6: MFR.Part INA180A2IDBVR -> (none); Manufacturing part number (none) -> INA180A2IDBVR; jlcpcb C192764 -> (none); jlcpcb part number (none) -> C192764

Commit message: [jlcpcb] Added gerbers, BOM, currently checking gerbers | TODO: Remove solder mask from larger pads
Parts:
- C1, C2, C3: value 0.47uF -> 470nF; footprint Capacitor_SMD:C_0805_2012Metric -> Capacitor_SMD:C_0603_1608Metric; LCSC Part Number (none) -> C1623; Manufacturing part number CL21A475KAQNNNE -> CL10B474KA8NNNC; jlcpcb part number C1779 -> (none)
- C10, C11, C12, C13, C14, C15, C7, C8, C9: LCSC Part Number (none) -> C15195; jlcpcb part number C15195 -> (none)
- C16, C17, C18: LCSC Part Number (none) -> C106666; jlcpcb part number C106666 -> (none)
- C19, C20, C21: LCSC Part Number (none) -> C307331; jlcpcb part number C307331 -> (none)
- C4, C5, C6: LCSC Part Number (none) -> C19666; jlcpcb part number C19666 -> (none)
- D1, D2, D3: LCSC Part Number (none) -> C191023; jlcpcb part number C191023 -> (none)
- Q1, Q2, Q3, Q4, Q5, Q6: LCSC Part Number (none) -> C2586; jlcpcb part number C2586 -> (none)
- R1, R2, R3: LCSC Part Number (none) -> C17903; jlcpcb part number C17903 -> (none)
- R10, R11, R12: LCSC Part Number (none) -> C500615; jlcpcb part number C500615 -> (none)
- R13, R14, R15, R16, R17, R18, R19, R20, R21: LCSC Part Number (none) -> C22936; jlcpcb part number C22936 -> (none)
- R22, R23, R24, R25, R26, R27, R28, R29, R30, R31, R32, R33: LCSC Part Number (none) -> C4216; jlcpcb part number C4216 -> (none)
- R4, R5, R6, R7, R8, R9: LCSC Part Number (none) -> C18019; jlcpcb part number C18019 -> (none)
- U1, U2, U3: LCSC Part Number (none) -> C5804631; jlcpcb part number C5804631 -> (none)
- U4, U5, U6: LCSC Part Number (none) -> C192764; jlcpcb part number C192764 -> (none)
