File: kicad/power.kicad_sch (KiCad schematic)
At the start: 54 parts, among them J4 TYPE-C-31-M-12, U10 MC34063AD, U11 MC34063AD, U12 XC6206P332MR-G, U13 TPS2116DRLR

Commit message: Exchanged button, 0.33 ohm resistor and 3-pin connectors with cheaper variants
Parts:
- C37, C39, C40, C41, C44, C45: MFR.Part CA55-B6R3M107T -> (none); Manufacturing part number (none) -> CA55-B6R3M107T; jlcpcb C568913 -> (none); jlcpcb part number (none) -> C568913
- C38, C46, C47: MFR.Part CL31B105KBHNNNE -> (none); Manufacturing part number (none) -> CL31B105KBHNNNE; jlcpcb C1848 -> (none); jlcpcb part number (none) -> C1848
- C42: MFR.Part 0805B471K500NT -> (none); Manufacturing part number (none) -> 0805B471K500NT; jlcpcb C1743 -> (none); jlcpcb part number (none) -> C1743
- C43: MFR.Part CL21B821KBANNNC -> (none); Manufacturing part number (none) -> CL21B821KBANNNC; jlcpcb C296722 -> (none); jlcpcb part number (none) -> C296722
- D4, D5: MFR.Part 1N5819WS -> (none); Manufacturing part number (none) -> 1N5819WS; jlcpcb C191023 -> (none); jlcpcb part number (none) -> C191023
- D6, D9: MFR.Part F.0603.00139/P2-0603R1TS2-06T-002 -> (none); Manufacturing part number (none) -> F.0603.00139/P2-0603R1TS2-06T-002; jlcpcb C7496820 -> (none); jlcpcb part number (none) -> C7496820
- D7: MFR.Part PRTR5V0U2X,215 -> (none); Manufacturing part number (none) -> PRTR5V0U2X,215; jlcpcb C12333 -> (none); jlcpcb part number (none) -> C12333
- F1, F2: MFR.Part BSMD1812-050-60V -> (none); Manufacturing part number (none) -> BSMD1812-050-60V; jlcpcb C883142 -> (none); jlcpcb part number (none) -> C883142
- J4: MFR.Part TYPE-C-31-M-12 -> (none); Manufacturing part number (none) -> TYPE-C-31-M-12; jlcpcb C165948 -> (none); jlcpcb part number (none) -> C165948
- L1, L2: MFR.Part SWPA6045S101MT -> (none); Manufacturing part number (none) -> SWPA6045S101MT; jlcpcb C60633 -> (none); jlcpcb part number (none) -> C60633
- R47: MFR.Part 0805W8F4701T5E -> (none); Manufacturing part number (none) -> 0805W8F4701T5E; jlcpcb C17673 -> (none); jlcpcb part number (none) -> C17673
- R48: MFR.Part 0603WAF1202T5E -> (none); Manufacturing part number (none) -> 0603WAF1202T5E; jlcpcb C22790 -> (none); jlcpcb part number (none) -> C22790
- R49, R50, R61, R62: MFR.Part 0603WAF3302T5E -> (none); Manufacturing part number (none) -> 0603WAF3302T5E; jlcpcb C4216 -> (none); jlcpcb part number (none) -> C4216
- R52, R53, R63: MFR.Part 0402WGF4990TCE -> (none); Manufacturing part number (none) -> 0402WGF4990TCE; jlcpcb C4125 -> (none); jlcpcb part number (none) -> C4125
- R54, R55: MFR.Part 0805W8F1501T5E -> (none); Manufacturing part number (none) -> 0805W8F1501T5E; jlcpcb C4310 -> (none); jlcpcb part number (none) -> C4310
- R56, R58: MFR.Part 0805W8F5101T5E -> (none); Manufacturing part number (none) -> 0805W8F5101T5E; jlcpcb C27834 -> (none); jlcpcb part number (none) -> C27834
- R59, R60: footprint Resistor_SMD:R_2512_6332Metric -> Resistor_SMD:R_1206_3216Metric; MFR.Part 25121WF330LT4E -> (none); Manufacturing part number (none) -> 1206W4J033KT5E; jlcpcb C25468 -> (none); jlcpcb part number (none) -> C25347
- U10, U11: MFR.Part MC34063 -> (none); Manufacturing part number (none) -> MC34063; jlcpcb C5349988 -> (none); jlcpcb part number (none) -> C5349988
- U12: MFR.Part XC6206P332MR-G -> (none); Manufacturing part number (none) -> XC6206P332MR-G; jlcpcb C5446 -> (none); jlcpcb part number (none) -> C5446
- U13: MFR.Part TPS2116DRLR -> (none); Manufacturing part number (none) -> TPS2116DRLR; jlcpcb C3235557 -> (none); jlcpcb part number (none) -> C3235557

Commit message: [jlcpcb] Added gerbers, BOM, currently checking gerbers | TODO: Remove solder mask from larger pads
Parts:
- C37, C39, C40, C41, C44, C45: LCSC Part Number (none) -> C568913; jlcpcb part number C568913 -> (none)
- C38, C46, C47: LCSC Part Number (none) -> C1848; jlcpcb part number C1848 -> (none)
- C42: footprint Capacitor_SMD:C_0805_2012Metric_Pad1.18x1.45mm_HandSolder -> Capacitor_SMD:C_0603_1608Metric; LCSC Part Number (none) -> C1620; Manufacturing part number 0805B471K500NT -> 0603B471K500NT; jlcpcb part number C1743 -> (none)
- C43: LCSC Part Number (none) -> C296722; jlcpcb part number C296722 -> (none)
- D4, D5: LCSC Part Number (none) -> C191023; jlcpcb part number C191023 -> (none)
- D6, D9: LCSC Part Number (none) -> C7496820; jlcpcb part number C7496820 -> (none)
- D7: LCSC Part Number (none) -> C12333; jlcpcb part number C12333 -> (none)
- F1, F2: LCSC Part Number (none) -> C883142; jlcpcb part number C883142 -> (none)
- J4: LCSC Part Number (none) -> C165948; jlcpcb part number C165948 -> (none)
- L1, L2: LCSC Part Number (none) -> C60633; jlcpcb part number C60633 -> (none)
- R47: LCSC Part Number (none) -> C17673; jlcpcb part number C17673 -> (none)
- R48: LCSC Part Number (none) -> C22790; jlcpcb part number C22790 -> (none)
- R49, R50, R61, R62: LCSC Part Number (none) -> C4216; jlcpcb part number C4216 -> (none)
- R52, R53, R63: LCSC Part Number (none) -> C4125; jlcpcb part number C4125 -> (none)
- R54, R55: LCSC Part Number (none) -> C4310; jlcpcb part number C4310 -> (none)
- R56, R58: LCSC Part Number (none) -> C27834; jlcpcb part number C27834 -> (none)
- R59, R60: LCSC Part Number (none) -> C25347; jlcpcb part number C25347 -> (none)
- U10, U11: LCSC Part Number (none) -> C5349988; jlcpcb part number C5349988 -> (none)
- U12: LCSC Part Number (none) -> C5446; jlcpcb part number C5446 -> (none)
- U13: LCSC Part Number (none) -> C3235557; jlcpcb part number C3235557 -> (none)
